File: eurorack-1u-output.kicad_pcb (KiCad board)
At the start: 2 copper layers, 18 parts, among them J1 Eurorack_Power_10pin_Unshroud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, U1 TL072, U2 TL072

Commit message: some progress
Parts:
- added D1: 1N4148WS, Diode_SMD:D_SOD-323, F.Cu at (106.8, 98.3)
- added D2: 1N4148WS, Diode_SMD:D_SOD-323, F.Cu at (106.8, 101.3)
- added D3: 1N4148WS, Diode_SMD:D_SOD-323, F.Cu at (106.8, 104.2)
- added D4: 1N4148WS, Diode_SMD:D_SOD-323, F.Cu at (106.8, 107.2)
- added D5: B140HW-7, Diode_SMD:D_SOD-123, F.Cu at (148.6, 79.4)
- added D6: B140HW-7, Diode_SMD:D_SOD-123, F.Cu at (146.8, 91.6)
- added L1: FerriteBead_0603_1.5A, Inductor_SMD:L_0603_1608Metric, F.Cu at (143.2, 79.4)
- added L2: FerriteBead_0603_1.5A, Inductor_SMD:L_0603_1608Metric, F.Cu at (141.8, 91.4)
- added POT1: output volume, PCM_4ms_Potentiometer:Potentiometer_Alps_RK09L_Double_Vertical, F.Cu at (121.3, 98.8)
- added POT2: headphones volume, PCM_4ms_Potentiometer:Potentiometer_Alps_RK09L_Double_Vertical, F.Cu at (97.3, 109.4)
- added R10: 10k, Resistor_SMD:R_0603_1608Metric, F.Cu at (88.9, 103.2)
- added R11: 75, Resistor_SMD:R_0603_1608Metric, F.Cu at (88.9, 105.7)
- added R12: 75, Resistor_SMD:R_0603_1608Metric, F.Cu at (88.9, 108.2)
- added R13: 10k, Resistor_SMD:R_0603_1608Metric, F.Cu at (88.9, 110.7)
- added R14: 10k, Resistor_SMD:R_0603_1608Metric, F.Cu at (88.9, 113.2)
- added R15: 75, Resistor_SMD:R_0603_1608Metric, F.Cu at (88.9, 115.7)
- added R16: 75, Resistor_SMD:R_0603_1608Metric, F.Cu at (88.9, 118.2)
- added R8: 100k, Resistor_SMD:R_0603_1608Metric, F.Cu at (82.0, 70.0)
- added R9: 10k, Resistor_SMD:R_0603_1608Metric, F.Cu at (88.9, 100.6)
- added U3: NE5532, Package_SO:SOIC-8_3.9x4.9mm_P1.27mm, F.Cu at (95.2, 122.8)
- added U4: NE5532, Package_SO:SOIC-8_3.9x4.9mm_P1.27mm, F.Cu at (103.2, 123.0)
- moved R2 38.3 mm to (80.6, 85.6)
- moved IN_R1 36.3 mm to (73.0, 75.7)
- moved IN_L1 31.7 mm to (73.0, 90.9)
- moved U1 17.0 mm to (87.7, 80.5)
- moved J1 14.0 mm to (155.7, 84.9)
- moved C2 5.48 mm to (95.4, 77.2), turned to -90 degrees
- moved C4 4.08 mm to (95.5, 84.4), turned to -90 degrees
Connections:
- C2 pad 2: unconnected-(C2-Pad2) -> /Pre-Headphones-L
- C3 pad 1: Net-(IN_R1-SIG) -> Net-(U1B--)
- C4 pad 2: unconnected-(C4-Pad2) -> /Pre-Headphones-R
- J1 pad 1: unconnected-(J1-+12V-Pad1) -> Net-(D5-A)
- J1 pad 10: unconnected-(J1--12V-Pad10) -> Net-(D6-K)
- J1 pad 2: unconnected-(J1-+12V-Pad2) -> Net-(D5-A)
- J1 pad 3: unconnected-(J1-GND-Pad3) -> GND
- J1 pad 4: unconnected-(J1-GND-Pad4) -> GND
- J1 pad 5: unconnected-(J1-GND-Pad5) -> GND
- J1 pad 6: unconnected-(J1-GND-Pad6) -> GND
- J1 pad 7: unconnected-(J1-GND-Pad7) -> GND
- J1 pad 8: unconnected-(J1-GND-Pad8) -> GND
- J1 pad 9: unconnected-(J1--12V-Pad9) -> Net-(D6-K)
- R3 pad 1: Net-(IN_R1-SIG) -> Net-(U1B--)
- R5 pad 1: unconnected-(R5-Pad1) -> Net-(POT1A-Center)
- R7 pad 1: unconnected-(R7-Pad1) -> Net-(POT1B-Center)
- U1 pad 4: unconnected-(U1C-V--Pad4) -> -12V
- U1 pad 6: Net-(IN_R1-SIG) -> Net-(U1B--)
- U1 pad 8: unconnected-(U1C-V+-Pad8) -> +12V
- U2 pad 4: unconnected-(U2C-V--Pad4) -> -12V
- U2 pad 8: unconnected-(U2C-V+-Pad8) -> +12V
